File: rodeurDeCables.sch (KiCad schematic (older format))
At the start: 23 parts, among them T1 2N2222, T2 2N2907, T3 2N2222, T4 2N2907, U1 NE555, U2 NE555

Commit message: adds some components
Parts:
- added J2, J? (x3): Conn_01x02, symbol Connector_Generic:Conn_01x02
- added R? (x5): 3k3, symbol Device:R
- added T? (x6): 2N2222, symbol Device:Q_NPN_BCE
- added T? (x6): 2N2907, symbol Device:Q_PNP_BCE
- BT1: symbol SparkFun-Batteries:BATTERY-9V -> rodeurDeCables-rescue:BATTERY-9V-SparkFun-Batteries
Connections:
- net GND: now also T2.2 (C), T4.2 (C), U?.11, U?.13, U?.5, U?.7 (Vss), U?.9, T?.2 (C), T?.2 (C), T?.2 (C), T?.2 (C), T?.2 (C), T?.2 (C)
- net VCC: now also T1.2 (C), T3.2 (C), U?.14 (Vdd), T?.2 (C), T?.2 (C), T?.2 (C), T?.2 (C), T?.2 (C), T?.2 (C)
- net at T1.1 (B): now also T2.1 (B), R?.1, T?.1 (B), T?.1 (B), T?.1 (B), T?.1 (B), T?.1 (B), T?.1 (B)
- net at T1.3 (E), T2.3 (E): now also R?.2
- net at U?.1: now also U2.3 (Q)
- net at U?.2: now also U?.3, R?.2
- net at T3.1 (B): now also T4.1 (B)
- net at T3.3 (E), T4.3 (E): now also J2.2 (Pin_2)
- new net: J2.1 (Pin_1), R?.1
- new net: R?.2, T?.3 (E), T?.3 (E) (x3)
- new net: T?.1 (B), T?.1 (B) (x3)
- new net: J?.2 (Pin_2), T?.3 (E), T?.3 (E) (x3)
- new net: J?.1 (Pin_1), R?.1 (x3)
Other:
- moved on the sheet: BT1, C1, C2, C3, C4, D1, R1, R2, R3, R4, R5, T1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
